File: KiCad/AuraView.kicad_sch (KiCad schematic)
At the start: 0 parts

Commit message: Created libraries
Other:
- added sheet Jaya (jaya.kicad_sch)
- added sheet Marcelo (marcelo.kicad_sch)
- added sheet Zachary (zachary.kicad_sch)
- note added: "Veuillez seulement editer le contenu de votre sheet et de vos symbol/footprint libraries"
Changed lines of the file:
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@@
 	(generator_version "9.0")
 	(paper "A4")
+	(text "Veuillez seulement editer le contenu de votre sheet et de vos symbol/footprint libraries"
+		(exclude_from_sim no)
+		(at 160.02 107.95 0)
+		(effects
+			(font
+				(size 1.27 1.27)
+			)
+		)
+	)
+	(sheet
+		(at 152.4 87.63)
+		(size 12.7 3.81)
+		(exclude_from_sim no)
+		(in_bom yes)
+		(on_board yes)
+		(dnp no)
+		(fields_autoplaced yes)
+		(stroke
+			(width 0.1524)
+			(type solid)
+		)
+		(fill
+			(color 0 0 0 0.0000)
+		)
+		(property "Sheetname" "Marcelo"
+			(at 152.4 86.9184 0)
+			(effects
+				(font
+					(size 1.27 1.27)
+				)
+				(justify left bottom)
+			)
+		)
+		(property "Sheetfile" "marcelo.kicad_sch"
+			(at 152.4 92.0246 0)
+			(effects
+				(font
+					(size 1.27 1.27)
+				)
+				(justify left top)
+			)
+		)
+		(instances
+			(project "AuraView"
+				(path "/bc06d563-4007-4b79-a2fd-3534d8dd4a5b"
+					(page "3")
+				)
+			)
+		)
+	)
+	(sheet
+		(at 127 87.63)
+		(size 12.7 3.81)
+		(exclude_from_sim no)
+		(in_bom yes)
+		(on_board yes)
+		(dnp no)
+		(fields_autoplaced yes)
+		(stroke
+			(width 0.1524)
+			(type solid)
+		)
+		(fill
+			(color 0 0 0 0.0000)
+		)
+		(property "Sheetname" "Jaya"
+			(at 127 86.9184 0)
+			(effects
+				(font
+					(size 1.27 1.27)
+				)
+				(justify left bottom)
+			)
+		)
+		(property "Sheetfile" "jaya.kicad_sch"
+			(at 127 92.0246 0)
+			(effects
+				(font
+					(size 1.27 1.27)
+				)
+				(justify left top)
+			)
+		)
+		(instances
+			(project "AuraView"
+				(path "/bc06d563-4007-4b79-a2fd-3534d8dd4a5b"
+					(page "4")
+				)
+			)
+		)
+	)
+	(sheet
+		(at 100.33 87.63)
+		(size 12.7 3.81)
+		(exclude_from_sim no)
+		(in_bom yes)
+		(on_board yes)
+		(dnp no)
+		(fields_autoplaced yes)
+		(stroke
+			(width 0.1524)
+			(type solid)
+		)
+		(fill
+			(color 0 0 0 0.0000)
+		)
+		(property "Sheetname" "Zachary"
+			(at 100.33 86.9184 0)
+			(effects
+				(font
+					(size 1.27 1.27)
+				)
+				(justify left bottom)
+			)
+		)
+		(property "Sheetfile" "zachary.kicad_sch"
+			(at 100.33 92.0246 0)
+			(effects
+				(font
+					(size 1.27 1.27)
+				)
+				(justify left top)
+			)
+		)
+		(instances
+			(project "AuraView"
+				(path "/bc06d563-4007-4b79-a2fd-3534d8dd4a5b"
+					(page "2")
+				)
+			)
+		)
+	)
 	(sheet_instances
 		(path "/"
