File: KiCad/zachary.kicad_sch (KiCad schematic)
At the start: 0 parts

Commit message: Zachary test
Other:
- note added: "THIS IS A TEST"
Changed lines of the file:
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@@
 	(generator_version "9.0")
 	(paper "A4")
+	(text "THIS IS A TEST"
+		(exclude_from_sim no)
+		(at 146.05 102.87 0)
+		(effects
+			(font
+				(size 1.27 1.27)
+			)
+		)
+	)
 )
