File: KiCad/jaya.kicad_sch (KiCad schematic)
At the start: 0 parts

Commit message: Jaya1
PSU (Inspired by CM4) and Motor Driver (not finished)
Other:
- added sheet Base (Base.kicad_sch)
- added sheet PCB (PCB.kicad_sch)
- note added: "Hollow Bore Slip-Ring + Motor"
- note added: "JAYA"
- note added: "MCU + Display Driver"
- note added: "Power Management + Motor Driver"
- note added: "Screen"
Changed lines of the file:
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@@
 	(generator_version "9.0")
 	(paper "A4")
+	(text "JAYA"
+		(exclude_from_sim no)
+		(at 17.018 14.986 0)
+		(effects
+			(font
+				(size 2.54 2.54)
+			)
+		)
+	)
+	(text "Screen"
+		(exclude_from_sim no)
+		(at 137.16 45.212 0)
+		(effects
+			(font
+				(size 2.54 2.54)
+			)
+		)
+	)
+	(text "Hollow Bore Slip-Ring + Motor"
+		(exclude_from_sim no)
+		(at 139.954 109.22 0)
+		(effects
+			(font
+				(size 1.27 1.27)
+			)
+		)
+	)
+	(text "Power Management + Motor Driver"
+		(exclude_from_sim no)
+		(at 143.764 153.162 0)
+		(effects
+			(font
+				(size 1.27 1.27)
+			)
+		)
+	)
+	(text "MCU + Display Driver"
+		(exclude_from_sim no)
+		(at 137.414 86.868 0)
+		(effects
+			(font
+				(size 1.27 1.27)
+			)
+		)
+	)
+	(sheet
+		(at 127 62.23)
+		(size 23.622 20.574)
+		(exclude_from_sim no)
+		(in_bom yes)
+		(on_board yes)
+		(dnp no)
+		(fields_autoplaced yes)
+		(stroke
+			(width 0.1524)
+			(type solid)
+		)
+		(fill
+			(color 0 0 0 0.0000)
+		)
+		(property "Sheetname" "PCB"
+			(at 127 61.5184 0)
+			(effects
+				(font
+					(size 1.27 1.27)
+				)
+				(justify left bottom)
+			)
+		)
+		(property "Sheetfile" "PCB.kicad_sch"
+			(at 127 83.3886 0)
+			(effects
+				(font
+					(size 1.27 1.27)
+				)
+				(justify left top)
+			)
+		)
+		(instances
+			(project "AuraView"
+				(path "/bc06d563-4007-4b79-a2fd-3534d8dd4a5b/4bf745a6-de54-4b83-90cc-a634239cb0a7"
+					(page "6")
+				)
+			)
+		)
+	)
+	(sheet
+		(at 127 128.27)
+		(size 23.368 21.336)
+		(exclude_from_sim no)
+		(in_bom yes)
+		(on_board yes)
+		(dnp no)
+		(fields_autoplaced yes)
+		(stroke
+			(width 0.1524)
+			(type solid)
+		)
+		(fill
+			(color 0 0 0 0.0000)
+		)
+		(property "Sheetname" "Base"
+			(at 127 127.5584 0)
+			(effects
+				(font
+					(size 1.27 1.27)
+				)
+				(justify left bottom)
+			)
+		)
+		(property "Sheetfile" "Base.kicad_sch"
+			(at 127 150.1906 0)
+			(effects
+				(font
+					(size 1.27 1.27)
+				)
+				(justify left top)
+			)
+		)
+		(instances
+			(project "AuraView"
+				(path "/bc06d563-4007-4b79-a2fd-3534d8dd4a5b/4bf745a6-de54-4b83-90cc-a634239cb0a7"
+					(page "5")
+				)
+			)
+		)
+	)
 )
